Commit message: feat: add iacquabot 3D models and update thruster configuration parameters

File: vrx_urdf/wamv_description/urdf/thrusters/engine.xacro (robot description, xacro)
@@ -4,8 +4,21 @@
   <xacro:macro name="engine" params="prefix position:='0 0 0' orientation:='0 0 0'">
     <link name="${namespace}/${prefix}_engine_link">
-      <visual>
+      <visual name="${prefix}_engine_housing_visual">
+        <origin xyz="-0.278156 0 -0.509371" rpy="0 0 0"/>
         <geometry>
-          <mesh filename="package://wamv_description/models/engine/mesh/engine.dae"/>
+          <mesh filename="package://vrx_gz/models/roboboat01/meshes/housing.dae" scale="0.7 0.7 0.7"/>
         </geometry>
+        <material name="pure_black">
+          <color rgba="0.0 0.0 0.0 1.0"/>
+        </material>
+      </visual>
+      <visual name="${prefix}_engine_mount_visual">
+        <origin xyz="-0.278156 0 -0.509371" rpy="0 0 0"/>
+        <geometry>
+          <mesh filename="package://vrx_gz/models/roboboat01/meshes/mount.dae" scale="0.7 0.7 0.7"/>
+        </geometry>
+        <material name="pure_black">
+          <color rgba="0.0 0.0 0.0 1.0"/>
+        </material>
       </visual>
       <collision name="${prefix}_engine_vertical_axis_collision">
@@ -22,13 +35,18 @@
       </collision>
       <inertial>
-        <mass value="15"/>
-        <inertia ixx="0.889245" ixy="0.0" ixz="0.0" iyy="0.911125" iyz="0.0" izz="0.078125"/>
+        <origin xyz="-0.278156 0 -0.409371" rpy="0 0 0"/>
+        <mass value="1.5"/>
+        <inertia ixx="0.088925" ixy="0.0" ixz="0.0" iyy="0.091112" iyz="0.0" izz="0.007812"/>
       </inertial>
     </link>
     <link name="${namespace}/${prefix}_propeller_link">
-      <visual>
+      <visual name="${prefix}_propeller_visual">
+        <origin xyz="0 0 0" rpy="0 0 0"/>
         <geometry>
-          <mesh filename="package://wamv_description/models/propeller/mesh/propeller.dae"/>
+          <mesh filename="package://vrx_gz/models/roboboat01/meshes/prop.dae" scale="0.7 0.7 0.7"/>
         </geometry>
+        <material name="orange_prop">
+          <color rgba="1.0 0.4 0.0 1.0"/>
+        </material>
       </visual>
       <collision name="${prefix}_propeller_collision">
@@ -39,6 +57,7 @@
       </collision>
       <inertial>
-        <mass value="0.5"/>
-        <inertia ixx="0.008545" ixy="0.0" ixz="0.0" iyy="0.008545" iyz="0.0" izz="0.0144"/>
+        <origin xyz="0 0 0" rpy="0 0 0"/>
+        <mass value="0.05"/>
+        <inertia ixx="0.000855" ixy="0.0" ixz="0.0" iyy="0.000855" iyz="0.0" izz="0.001440"/>
       </inertial>
     </link>
@@ -58,4 +77,28 @@
       <dynamics friction="0.05" damping="0.05" />
     </joint>
+    <gazebo reference="${namespace}/${prefix}_engine_link">
+      <visual>
+        <material>
+          <ambient>0.005 0.005 0.005 1.0</ambient>
+          <diffuse>0.01 0.01 0.01 1.0</diffuse>
+          <specular>0.3 0.3 0.3 1.0</specular>
+          <pbr>
+            <metal>
+              <roughness>0.3</roughness>
+              <metalness>0.5</metalness>
+            </metal>
+          </pbr>
+        </material>
+      </visual>
+    </gazebo>
+    <gazebo reference="${namespace}/${prefix}_propeller_link">
+      <visual>
+        <material>
+          <ambient>0.9 0.35 0.0 1.0</ambient>
+          <diffuse>1.0 0.4 0.0 1.0</diffuse>
+          <specular>0.5 0.5 0.5 1.0</specular>
+        </material>
+      </visual>
+    </gazebo>
   </xacro:macro>
 </robot>

File: vrx_urdf/wamv_description/urdf/wamv_base.urdf.xacro (robot description, xacro)
@@ -87,12 +87,10 @@
   <link name="${namespace}/base_link">
     <!-- Main base hull (base.glb) -->
-    <visual name="base_visual">
+    <!-- Main base hull (base.glb) -->
+    <visual>
       <origin xyz="0 0 0.05" rpy="1.5708 0 3.14159"/>
       <geometry>
         <mesh filename="package://wamv_description/models/iacquabot_model/base.glb" scale="1.15 1.15 1.15"/>
       </geometry>
-      <material name="iacquabot_green">
-        <color rgba="0.18039 0.49020 0.19608 1.0"/>
-      </material>
     </visual>
     <!-- Left base collisions -->
@@ -115,12 +113,9 @@
   <!-- Front Bow (proa.STL) as separate link for PBR metallic material support -->
   <link name="${namespace}/proa_link">
-    <visual name="proa_visual">
+    <visual>
       <origin xyz="0 0 0" rpy="1.5708 0 1.5708"/>
       <geometry>
         <mesh filename="package://wamv_description/models/iacquabot_model/proa.STL" scale="0.001 0.001 0.001"/>
       </geometry>
-      <material name="iacquabot_dark_blue">
-        <color rgba="0.015 0.065 0.320 1.0"/>
-      </material>
     </visual>
   </link>
@@ -129,4 +124,18 @@
     <parent link="${namespace}/base_link"/>
     <child link="${namespace}/proa_link"/>
+  </joint>
+  <!-- Decal Link attached to Tablet (Logo & Name) -->
+  <link name="${namespace}/deck_decal_link">
+    <visual>
+      <origin xyz="0 0 0" rpy="0 0 0"/>
+      <geometry>
+        <box size="0.118 0.168 0.002"/>
+      </geometry>
+    </visual>
+  </link>
+  <joint name="${namespace}/deck_decal_joint" type="fixed">
+    <origin xyz="0.0 0.01 -0.015" rpy="0 0 3.14159"/>
+    <parent link="${namespace}/tablet_link"/>
+    <child link="${namespace}/deck_decal_link"/>
   </joint>
   <gazebo>
@@ -138,5 +147,11 @@
         <ambient>0.18039 0.49020 0.19608 1.0</ambient>
         <diffuse>0.18039 0.49020 0.19608 1.0</diffuse>
-        <specular>0.5 0.5 0.5 1.0</specular>
+        <specular>0.6 0.6 0.6 1.0</specular>
+        <pbr>
+          <metal>
+            <roughness>0.3</roughness>
+            <metalness>0.3</metalness>
+          </metal>
+        </pbr>
       </material>
     </visual>
@@ -162,9 +177,9 @@
         <ambient>0.015 0.065 0.320 1.0</ambient>
         <diffuse>0.015 0.065 0.320 1.0</diffuse>
-        <specular>1.0 1.0 1.0 1.0</specular>
+        <specular>0.6 0.6 0.6 1.0</specular>
         <pbr>
           <metal>
-            <roughness>0.15</roughness>
-            <metalness>0.9</metalness>
+            <roughness>0.3</roughness>
+            <metalness>0.3</metalness>
           </metal>
         </pbr>
@@ -172,3 +187,77 @@
     </visual>
   </gazebo>
+  <gazebo reference="${namespace}/deck_decal_link">
+    <visual>
+      <material>
+        <ambient>1.0 1.0 1.0 1.0</ambient>
+        <diffuse>1.0 1.0 1.0 1.0</diffuse>
+        <specular>0.3 0.3 0.3 1.0</specular>
+        <pbr>
+          <metal>
+            <albedo_map>model://wamv_description/models/iacquabot_model/iacquabot_deck_decal.png</albedo_map>
+            <roughness>0.3</roughness>
+            <metalness>0.0</metalness>
+          </metal>
+        </pbr>
+      </material>
+    </visual>
+  </gazebo>
+  <!-- Tablet Link (15cm in front of camera: X=0.45, Y=0.0, Z=0.17, scale=0.096, pitch=230 deg) -->
+  <link name="${namespace}/tablet_link">
+    <visual>
+      <origin xyz="0 0 0" rpy="1.5708 0 1.5708"/>
+      <geometry>
+        <mesh filename="package://wamv_description/models/iacquabot_model/tablet/scene.gltf" scale="0.096 0.096 0.096"/>
+      </geometry>
+    </visual>
+  </link>
+  <joint name="${namespace}/tablet_joint" type="fixed">
+    <origin xyz="0.45 0.0 0.17" rpy="0 4.01426 0"/>
+    <parent link="${namespace}/base_link"/>
+    <child link="${namespace}/tablet_link"/>
+  </joint>
+  <link name="${namespace}/solar_panel_link">
+    <visual>
+      <origin xyz="0 2.5811 -0.1142" rpy="-1.5708 0 -1.5708"/>
+      <geometry>
+        <mesh filename="package://wamv_description/models/iacquabot_model/solar_panel/scene.gltf" scale="0.01235 0.00855 0.0095"/>
+      </geometry>
+    </visual>
+  </link>
+  <joint name="${namespace}/solar_panel_joint" type="fixed">
+    <origin xyz="-0.10 0.0 0.12" rpy="0 0 0"/>
+    <parent link="${namespace}/base_link"/>
+    <child link="${namespace}/solar_panel_link"/>
+  </joint>
+  <!-- Gray Pole Link (Diameter: 1.5cm, Height: 50cm, 8cm next to camera) -->
+  <link name="${namespace}/camera_pole_link">
+    <visual>
+      <origin xyz="0 0 0" rpy="0 0 0"/>
+      <geometry>
+        <cylinder radius="0.0075" length="0.50"/>
+      </geometry>
+      <material name="gray_pole_mat">
+        <color rgba="0.5 0.5 0.5 1.0"/>
+      </material>
+    </visual>
+  </link>
+  <joint name="${namespace}/camera_pole_joint" type="fixed">
+    <origin xyz="0.30 0.08 0.33" rpy="0 0 0"/>
+    <parent link="${namespace}/base_link"/>
+    <child link="${namespace}/camera_pole_link"/>
+  </joint>
+  <!-- Router Link (Mounted on camera pole, 0.9x narrower, 1.5x taller, face forward) -->
+  <link name="${namespace}/router_link">
+    <visual>
+      <origin xyz="0 0 0" rpy="0 0 3.14159"/>
+      <geometry>
+        <mesh filename="package://wamv_description/models/iacquabot_model/modelrouter/scene.gltf" scale="1.0 0.9 1.5"/>
+      </geometry>
+    </visual>
+  </link>
+  <joint name="${namespace}/router_joint" type="fixed">
+    <origin xyz="0.03 0.0 0.15" rpy="0 0 0"/>
+    <parent link="${namespace}/camera_pole_link"/>
+    <child link="${namespace}/router_link"/>
+  </joint>
 </robot>

File: vrx_urdf/wamv_gazebo/urdf/thruster_layouts/wamv_aft_thrusters.xacro (robot description, xacro)
@@ -2,6 +2,6 @@
 <robot xmlns:xacro="http://ros.org/wiki/xacro">
   <xacro:include filename="$(find wamv_description)/urdf/thrusters/engine.xacro" />
-  <xacro:engine prefix="left" position="-2.373776 1.027135 0.318237" />
-  <xacro:engine prefix="right" position="-2.373776 -1.027135 0.318237" />
+  <xacro:engine prefix="left" position="-0.10 0.20 0.468237" />
+  <xacro:engine prefix="right" position="-0.10 -0.20 0.468237" />
   <xacro:include filename="$(find wamv_gazebo)/urdf/thruster_layouts/wamv_gazebo_thruster_config.xacro" />
   <xacro:wamv_gazebo_thruster_config name="left" />

File: vrx_urdf/wamv_gazebo/urdf/thruster_layouts/wamv_t_thrusters.xacro (robot description, xacro)
@@ -2,7 +2,7 @@
 <robot xmlns:xacro="http://ros.org/wiki/xacro">
   <xacro:include filename="$(find wamv_description)/urdf/thrusters/engine.xacro" />
-  <xacro:engine prefix="left" position="-2.373776 1.027135 0.318237" />
-  <xacro:engine prefix="right" position="-2.373776 -1.027135 0.318237" />
-  <xacro:engine prefix="lateral" position="0.0 0.0 0.318237" orientation="0.0 0.0 1.5707"/>
+  <xacro:engine prefix="left" position="-0.10 0.20 0.468237" />
+  <xacro:engine prefix="right" position="-0.10 -0.20 0.468237" />
+  <xacro:engine prefix="lateral" position="0.60 0.0 0.468237" orientation="0.0 0.0 1.5707"/>
   <xacro:include filename="$(find wamv_gazebo)/urdf/thruster_layouts/wamv_gazebo_thruster_config.xacro" />
   <xacro:wamv_gazebo_thruster_config name="left" />

File: vrx_urdf/wamv_gazebo/urdf/thruster_layouts/wamv_x_thrusters.xacro (robot description, xacro)
@@ -2,8 +2,8 @@
 <robot xmlns:xacro="http://ros.org/wiki/xacro">
   <xacro:include filename="$(find wamv_description)/urdf/thrusters/engine.xacro" />
-  <xacro:engine prefix="left_rear" position="-2.373776 1.027135 0.318237"  orientation="0.0 0.0 0.0"/>
-  <xacro:engine prefix="right_rear" position="-2.373776 -1.027135 0.318237" orientation="0.0 0.0 0.0"/>
-  <xacro:engine prefix="left_front" position="1.6 1.027135 0.318237" orientation="0.0 0.0 0.0"/>
-  <xacro:engine prefix="right_front" position="1.6 -1.027135 0.318237" orientation="0.0 0.0 0.0"/>
+  <xacro:engine prefix="left_rear" position="-0.10 0.20 0.468237" orientation="0.0 0.0 0.0"/>
+  <xacro:engine prefix="right_rear" position="-0.10 -0.20 0.468237" orientation="0.0 0.0 0.0"/>
+  <xacro:engine prefix="left_front" position="0.60 0.20 0.468237" orientation="0.0 0.0 0.0"/>
+  <xacro:engine prefix="right_front" position="0.60 -0.20 0.468237" orientation="0.0 0.0 0.0"/>
   <xacro:include filename="$(find wamv_gazebo)/urdf/thruster_layouts/wamv_gazebo_thruster_config.xacro" />
   <xacro:wamv_gazebo_thruster_config name="left_rear" />
