Commit message: identification vrx

File: vrx_urdf/wamv_description/urdf/thrusters/engine.xacro (robot description, xacro)
@@ -1,5 +1,4 @@
 <?xml version="1.0"?>
 <robot xmlns:xacro="http://ros.org/wiki/xacro" name="wam-v-two-engines">
-  <!-- Macro for inserting an engine with its propeller. -->
   <xacro:macro name="engine" params="prefix position:='0 0 0' orientation:='0 0 0'">
     <link name="${namespace}/${prefix}_engine_link">
@@ -7,5 +6,5 @@
         <origin xyz="-0.278156 0 -0.509371" rpy="0 0 0"/>
         <geometry>
-          <mesh filename="package://vrx_gz/models/roboboat01/meshes/housing.dae" scale="0.7 0.7 0.7"/>
+          <mesh filename="package://vrx_gz/models/roboboat01/meshes/housing.dae" scale="1.0 1.0 1.0"/>
         </geometry>
         <material name="pure_black">
@@ -16,5 +15,5 @@
         <origin xyz="-0.278156 0 -0.509371" rpy="0 0 0"/>
         <geometry>
-          <mesh filename="package://vrx_gz/models/roboboat01/meshes/mount.dae" scale="0.7 0.7 0.7"/>
+          <mesh filename="package://vrx_gz/models/roboboat01/meshes/mount.dae" scale="1.0 1.0 1.0"/>
         </geometry>
         <material name="pure_black">
@@ -25,5 +24,5 @@
         <origin xyz="-0.16 0 -0.24" rpy="0 0 0" />
         <geometry>
-          <box size="0.2 0.15 0.83" />
+          <box size="0.2 0.15 1.03" />
         </geometry>
       </collision>
@@ -34,8 +33,10 @@
         </geometry>
       </collision>
+      <!-- Masa real del T200 (0.344 kg), pero inercia con piso numérico
+           razonable para que el solver no se vuelva inestable/degenerado. -->
       <inertial>
         <origin xyz="-0.278156 0 -0.409371" rpy="0 0 0"/>
-        <mass value="1.5"/>
-        <inertia ixx="0.088925" ixy="0.0" ixz="0.0" iyy="0.091112" iyz="0.0" izz="0.007812"/>
+        <mass value="0.344"/>
+        <inertia ixx="0.005" ixy="0.0" ixz="0.0" iyy="0.005" iyz="0.0" izz="0.002"/>
       </inertial>
     </link>
@@ -44,5 +45,5 @@
         <origin xyz="0 0 0" rpy="0 0 0"/>
         <geometry>
-          <mesh filename="package://vrx_gz/models/roboboat01/meshes/prop.dae" scale="0.7 0.7 0.7"/>
+          <mesh filename="package://vrx_gz/models/roboboat01/meshes/prop.dae" scale="1.0 1.0 1.0"/>
         </geometry>
         <material name="orange_prop">
@@ -56,8 +57,10 @@
         </geometry>
       </collision>
+      <!-- Masa real de la hélice (0.012 kg), inercia con piso numérico
+           (no la real de ~1e-6, que hacía fallar al solver del joint continuo). -->
       <inertial>
         <origin xyz="0 0 0" rpy="0 0 0"/>
-        <mass value="0.05"/>
-        <inertia ixx="0.000855" ixy="0.0" ixz="0.0" iyy="0.000855" iyz="0.0" izz="0.001440"/>
+        <mass value="0.012"/>
+        <inertia ixx="0.0005" ixy="0.0" ixz="0.0" iyy="0.0005" iyz="0.0" izz="0.0003"/>
       </inertial>
     </link>

File: vrx_urdf/wamv_description/urdf/wamv_base.urdf.xacro (robot description, xacro)
@@ -76,5 +76,4 @@
       </geometry>
     </collision>
-    <!-- Joint -->
     <collision name="${prefix}_joint">
       <origin xyz="0.58 ${1.03*reflect} 0.6" rpy="${0*reflect} -0.6 0" />
@@ -84,12 +83,9 @@
     </collision>
   </xacro:macro>
-  <!-- Basic model of the 16' WAM-V USV -->
   <link name="${namespace}/base_link">
-    <!-- Main base hull (base.glb) -->
-    <!-- Main base hull (base.glb) -->
     <visual>
       <origin xyz="0 0 0.05" rpy="1.5708 0 3.14159"/>
       <geometry>
-        <mesh filename="package://wamv_description/models/iacquabot_model/base.glb" scale="1.15 1.15 1.15"/>
+        <mesh filename="package://wamv_description/models/iacquabot_model/base.glb" scale="1.4 1.12 1.55"/>
       </geometry>
     </visual>
@@ -110,15 +106,14 @@
 </inertial>
   </link>
-  <!-- Front Bow (proa.STL) as separate link for PBR metallic material support -->
   <link name="${namespace}/proa_link">
     <visual>
       <origin xyz="0 0 0" rpy="1.5708 0 1.5708"/>
       <geometry>
-        <mesh filename="package://wamv_description/models/iacquabot_model/proa.STL" scale="0.001 0.001 0.001"/>
+        <mesh filename="package://wamv_description/models/iacquabot_model/proa.STL" scale="0.0013 0.0013 0.0013"/>
       </geometry>
     </visual>
   </link>
   <joint name="${namespace}/proa_joint" type="fixed">
-    <origin xyz="0.40 -0.22368 -0.02" rpy="0 0 0"/>
+    <origin xyz="0.45 -0.27368 -0.065" rpy="0 0 0"/>
     <parent link="${namespace}/base_link"/>
     <child link="${namespace}/proa_link"/>
@@ -129,10 +124,10 @@
       <origin xyz="0 0 0" rpy="0 0 0"/>
       <geometry>
-        <box size="0.118 0.168 0.002"/>
+        <box size="0.15 0.25 0.002"/>
       </geometry>
     </visual>
   </link>
   <joint name="${namespace}/deck_decal_joint" type="fixed">
-    <origin xyz="0.0 0.01 -0.015" rpy="0 0 3.14159"/>
+    <origin xyz="0.0 0.01 -0.02" rpy="0 0 3.14159"/>
     <parent link="${namespace}/tablet_link"/>
     <child link="${namespace}/deck_decal_link"/>
@@ -207,10 +202,10 @@
       <origin xyz="0 0 0" rpy="1.5708 0 1.5708"/>
       <geometry>
-        <mesh filename="package://wamv_description/models/iacquabot_model/tablet/scene.gltf" scale="0.096 0.096 0.096"/>
+        <mesh filename="package://wamv_description/models/iacquabot_model/tablet/scene.gltf" scale="0.14 0.14 0.14"/>
       </geometry>
     </visual>
   </link>
   <joint name="${namespace}/tablet_joint" type="fixed">
-    <origin xyz="0.45 0.0 0.17" rpy="0 4.01426 0"/>
+    <origin xyz="0.55 0.0 0.182" rpy="0 4.01426 0"/>
     <parent link="${namespace}/base_link"/>
     <child link="${namespace}/tablet_link"/>
@@ -218,7 +213,7 @@
   <link name="${namespace}/solar_panel_link">
     <visual>
-      <origin xyz="0 2.5811 -0.1142" rpy="-1.5708 0 -1.5708"/>
-      <geometry>
-        <mesh filename="package://wamv_description/models/iacquabot_model/solar_panel/scene.gltf" scale="0.01235 0.00855 0.0095"/>
+      <origin xyz="-0.0 3.4 -0.13" rpy="-1.5708 0 -1.5708"/>
+      <geometry>
+        <mesh filename="package://wamv_description/models/iacquabot_model/solar_panel/scene.gltf" scale="0.0162 0.01 0.011"/>
       </geometry>
     </visual>
@@ -229,5 +224,4 @@
     <child link="${namespace}/solar_panel_link"/>
   </joint>
-  <!-- Gray Pole Link (Diameter: 1.5cm, Height: 50cm, 8cm next to camera) -->
   <link name="${namespace}/camera_pole_link">
     <visual>
@@ -242,5 +236,5 @@
   </link>
   <joint name="${namespace}/camera_pole_joint" type="fixed">
-    <origin xyz="0.30 0.08 0.33" rpy="0 0 0"/>
+    <origin xyz="0.35 0.09 0.33" rpy="0 0 0"/>
     <parent link="${namespace}/base_link"/>
     <child link="${namespace}/camera_pole_link"/>
@@ -251,10 +245,10 @@
       <origin xyz="0 0 0" rpy="0 0 3.14159"/>
       <geometry>
-        <mesh filename="package://wamv_description/models/iacquabot_model/modelrouter/scene.gltf" scale="1.0 0.9 1.5"/>
+        <mesh filename="package://wamv_description/models/iacquabot_model/modelrouter/scene.gltf" scale="1.3 1.1 2.5"/>
       </geometry>
     </visual>
   </link>
   <joint name="${namespace}/router_joint" type="fixed">
-    <origin xyz="0.03 0.0 0.15" rpy="0 0 0"/>
+    <origin xyz="0.035 0.0 0.25" rpy="0 0 0"/>
     <parent link="${namespace}/camera_pole_link"/>
     <child link="${namespace}/router_link"/>

File: vrx_urdf/wamv_gazebo/urdf/dynamics/wamv_gazebo_dynamics_plugin.xacro (robot description, xacro)
@@ -4,5 +4,5 @@
     <!--Gazebo Plugin for simulating board dynamics-->
     <gazebo>
-      <!-- Left hull -->
+      <!-- Lado izquierdo -->
       <plugin
         filename="libSurface.so"
@@ -10,9 +10,10 @@
         <link_name>${namespace}/base_link</link_name>
         <hull_length>1.2</hull_length>
-        <hull_radius>0.15</hull_radius>
+        <hull_radius>0.25</hull_radius>
         <fluid_level>0</fluid_level>
         <points>
-          <point>0.6 0.169 0</point>
-          <point>-0.6 0.169 0</point>
+          <point>0.55  0.25 0</point>
+          <point>0.0   0.25 0</point>
+          <point>-0.55 0.25 0</point>
         </points>
         <wavefield>
@@ -20,5 +21,6 @@
         </wavefield>
       </plugin>
-      <!-- Right hull -->
+      <!-- Lado derecho (corregido: antes estaba en 0.169, asimétrico respecto
+           al izquierdo en 0.25 — esa asimetría causaba roll constante) -->
       <plugin
         filename="libSurface.so"
@@ -26,9 +28,10 @@
         <link_name>${namespace}/base_link</link_name>
         <hull_length>1.2</hull_length>
-        <hull_radius>0.15</hull_radius>
+        <hull_radius>0.25</hull_radius>
         <fluid_level>0</fluid_level>
         <points>
-          <point>0.6 -0.169 0</point>
-          <point>-0.6 -0.169 0</point>
+          <point>0.55  -0.25 0</point>
+          <point>0.0   -0.25 0</point>
+          <point>-0.55 -0.25 0</point>
         </points>
         <wavefield>
@@ -36,25 +39,22 @@
         </wavefield>
       </plugin>
-    <plugin
-        filename="libSimpleHydrodynamics.so"
-        name="vrx::SimpleHydrodynamics">
-        <link_name>${namespace}/base_link</link_name>
-        <!-- Added mass -->
-        <xDotU>2.85</xDotU>
-        <yDotV>8.36</yDotV>
-        <nDotR>2.34</nDotR>
-        <!-- Arrastres Lineales y Cuadráticos Optimizados -->
-        <xU>13.91</xU>
-        <xUU>14.92</xUU>
-        <yV>49.04</yV>
-        <yVV>1.01</yVV>
-        <nR>6.03</nR>
-        <nRR>2.91</nRR>
-        <!-- ESTOS ERAN LOS CULPABLES (Bájalos drásticamente) -->
-        <zW>20.0</zW>    <!-- Fricción vertical (Heave) -->
-        <kP>2.0</kP>     <!-- Fricción de balanceo (Roll) -->
-        <kPP>2.0</kPP>
-        <mQ>5.0</mQ>     <!-- Fricción de cabeceo (Pitch) -->
-        <mQQ>5.0</mQQ>
+      <plugin
+          filename="libSimpleHydrodynamics.so"
+          name="vrx::SimpleHydrodynamics">
+          <link_name>${namespace}/base_link</link_name>
+          <xDotU>2.85</xDotU>
+          <yDotV>8.36</yDotV>
+          <nDotR>1.957</nDotR>
+          <xU>13.91</xU>
+          <xUU>14.92</xUU>
+          <yV>49.04</yV>
+          <yVV>1.01</yVV>
+          <nR>6.03</nR>
+          <nRR>2.91</nRR>
+          <zW>60.0</zW>
+          <kP>8.0</kP>
+          <kPP>8.0</kPP>
+          <mQ>2.0</mQ>
+          <mQQ>2.0</mQQ>
       </plugin>
     </gazebo>

File: vrx_urdf/wamv_gazebo/urdf/thruster_layouts/wamv_gazebo_thruster_config.xacro (robot description, xacro)
@@ -1,14 +1,10 @@
 <?xml version="1.0"?>
 <plugin xmlns:xacro="http://ros.org/wiki/xacro">
-  <xacro:macro  name="wamv_gazebo_thruster_config" params="name">
+  <xacro:macro name="wamv_gazebo_thruster_config" params="name">
   <gazebo>
-    <xacro:property name="x_uu" value="72.4" />
-    <xacro:property name="x_u" value="51.3" />
-    <xacro:property name="max_velocity_mps" value="7.71667" />
     <plugin
       filename="gz-sim-thruster-system"
       name="gz::sim::systems::Thruster">
       <joint_name>${namespace}/${name}_engine_propeller_joint</joint_name>
-      <!-- Empirical and physical parameters of the BlueRobotics T200 Thruster -->
       <cmd_timeout>0.5</cmd_timeout>
       <thrust_coefficient>0.1079</thrust_coefficient>
@@ -19,5 +15,4 @@
       <namespace>${namespace}</namespace>
       <topic>thrusters/${name}/thrust</topic>
-      <!-- Not used by Gazebo but used to run the bridge easily -->
       <name>${name}</name>
     </plugin>
@@ -28,5 +23,4 @@
       <use_velocity_commands>true</use_velocity_commands>
       <topic>${namespace}/thrusters/${name}/pos</topic>
-      <!-- Not used by Gazebo but used to run the bridge easily -->
       <name>${name}</name>
     </plugin>

File: vrx_urdf/wamv_gazebo/urdf/thruster_layouts/wamv_x_thrusters.xacro (robot description, xacro)
@@ -2,8 +2,8 @@
 <robot xmlns:xacro="http://ros.org/wiki/xacro">
   <xacro:include filename="$(find wamv_description)/urdf/thrusters/engine.xacro" />
-  <xacro:engine prefix="left_rear" position="-0.10 0.20 0.468237" orientation="0.0 0.0 0.0"/>
-  <xacro:engine prefix="right_rear" position="-0.10 -0.20 0.468237" orientation="0.0 0.0 0.0"/>
-  <xacro:engine prefix="left_front" position="0.60 0.20 0.468237" orientation="0.0 0.0 0.0"/>
-  <xacro:engine prefix="right_front" position="0.60 -0.20 0.468237" orientation="0.0 0.0 0.0"/>
+  <xacro:engine prefix="left_rear"   position="-0.15  0.29 0.468237" orientation="0.0 0.0 0.0"/>
+  <xacro:engine prefix="right_rear"  position="-0.15 -0.29 0.468237" orientation="0.0 0.0 0.0"/>
+  <xacro:engine prefix="left_front"  position=" 0.60  0.29 0.468237" orientation="0.0 0.0 0.0"/>
+  <xacro:engine prefix="right_front" position=" 0.60 -0.29 0.468237" orientation="0.0 0.0 0.0"/>
   <xacro:include filename="$(find wamv_gazebo)/urdf/thruster_layouts/wamv_gazebo_thruster_config.xacro" />
   <xacro:wamv_gazebo_thruster_config name="left_rear" />

File: vrx_urdf/wamv_gazebo/urdf/wamv_gazebo.urdf.xacro (robot description, xacro)
@@ -106,5 +106,5 @@
     <!-- Add a front camera -->
     <xacro:if value="$(arg camera_enabled)">
-      <xacro:wamv_camera name="front_camera" x="0.30" y="0.0" z="0.40" post_z_from="0.05" P="${radians(15)}" />
+      <xacro:wamv_camera name="front_camera" x="0.42" y="0.0" z="0.40" post_z_from="0.05" P="${radians(15)}" />
     </xacro:if>
     <!-- Add simulated GPS -->
