Commit message: Alineación de propulsores delanteros y traseros a y=1.027

File: vrx_urdf/wamv_description/urdf/wamv_base.urdf.xacro (robot description, xacro)
@@ -103,7 +103,7 @@
     </collision>
     <inertial>
-      <!-- From WAM-V spec sheet -->
-      <mass value="180.0"/>
-      <inertia ixx="120.0" ixy="0.0" ixz="0.0" iyy="393" iyz="0.0" izz="446.0"/>
+      <!-- Customized WAM-V base values from user -->
+      <mass value="24.0"/>
+      <inertia ixx="4.77" ixy="0.0" ixz="0.0" iyy="1.01" iyz="0.0" izz="5.78"/>
     </inertial>
   </link>

File: vrx_urdf/wamv_gazebo/urdf/components/wamv_p3d.xacro (robot description, xacro)
@@ -7,5 +7,5 @@
         name="gz::sim::systems::OdometryPublisher">
         <dimensions>3</dimensions>
-        <odom_publish_frequency>10.0</odom_publish_frequency>
+        <odom_publish_frequency>30.0</odom_publish_frequency>
         <odom_frame>map</odom_frame>
         <robot_base_frame>wamv/base_link</robot_base_frame>

File: vrx_urdf/wamv_gazebo/urdf/dynamics/wamv_gazebo_dynamics_plugin.xacro (robot description, xacro)
@@ -45,15 +45,15 @@
         <nDotR>0.0</nDotR>
         <!-- Linear and quadratic drag -->
-        <xU>100.0</xU>
-        <xUU>150.0</xUU>
-        <yV>100.0</yV>
-        <yVV>100.0</yVV>
+        <xU>23.0</xU>
+        <xUU>38.0</xUU>
+        <yV>40.0</yV>
+        <yVV>30.0</yVV>
         <zW>500.0</zW>
-        <kP>300.0</kP>
-        <kPP>600.0</kPP>
-        <mQ>900.0</mQ>
-        <mQQ>900.0</mQQ>
-        <nR>800.0</nR>
-        <nRR>800.0</nRR>
+        <kP>100.0</kP>
+        <kPP>100.0</kPP>
+        <mQ>100.0</mQ>
+        <mQQ>100.0</mQQ>
+        <nR>100.0</nR>
+        <nRR>10.0</nRR>
       </plugin>
     </gazebo>

File: vrx_urdf/wamv_gazebo/urdf/thruster_layouts/wamv_gazebo_thruster_config.xacro (robot description, xacro)
@@ -10,10 +10,10 @@
       name="gz::sim::systems::Thruster">
       <joint_name>${namespace}/${name}_engine_propeller_joint</joint_name>
-      <thrust_coefficient>0.004422</thrust_coefficient>
+      <!-- Empirical and physical parameters of the BlueRobotics T200 Thruster -->
+      <thrust_coefficient>0.1079</thrust_coefficient>
       <fluid_density>1000</fluid_density>
-      <propeller_diameter>0.2</propeller_diameter>
-      <velocity_control>true</velocity_control>
-      <!-- max total thrust / 2 -->
-      <max_thrust_cmd>${((x_u + x_uu * max_velocity_mps) * max_velocity_mps)/ 2}</max_thrust_cmd>
+      <propeller_diameter>0.0762</propeller_diameter>
+      <velocity_control>false</velocity_control>
+      <max_thrust_cmd>36.3827</max_thrust_cmd>
       <namespace>${namespace}</namespace>
       <topic>thrusters/${name}/thrust</topic>

File: vrx_urdf/wamv_gazebo/urdf/thruster_layouts/wamv_x_thrusters.xacro (robot description, xacro)
@@ -2,8 +2,8 @@
 <robot xmlns:xacro="http://ros.org/wiki/xacro">
   <xacro:include filename="$(find wamv_description)/urdf/thrusters/engine.xacro" />
-  <xacro:engine prefix="left_rear" position="-2.373776 1.027135 0.318237"  orientation="0.0 0.0 0.785"/>
-  <xacro:engine prefix="right_rear" position="-2.373776 -1.027135 0.318237" orientation="0.0 0.0 -0.785"/>
-  <xacro:engine prefix="left_front" position="1.6 0.7  0.25" orientation="0.0 0.0 -0.785"/>
-  <xacro:engine prefix="right_front" position="1.6 -0.7 0.25" orientation="0.0 0.0 +0.785"/>
+  <xacro:engine prefix="left_rear" position="-2.373776 1.027135 0.318237"  orientation="0.0 0.0 0.0"/>
+  <xacro:engine prefix="right_rear" position="-2.373776 -1.027135 0.318237" orientation="0.0 0.0 0.0"/>
+  <xacro:engine prefix="left_front" position="1.6 1.027135 0.318237" orientation="0.0 0.0 0.0"/>
+  <xacro:engine prefix="right_front" position="1.6 -1.027135 0.318237" orientation="0.0 0.0 0.0"/>
   <xacro:include filename="$(find wamv_gazebo)/urdf/thruster_layouts/wamv_gazebo_thruster_config.xacro" />
   <xacro:wamv_gazebo_thruster_config name="left_rear" />

File: vrx_urdf/wamv_gazebo/urdf/wamv_gazebo.urdf.xacro (robot description, xacro)
@@ -37,7 +37,9 @@
   <xacro:include filename="$(find wamv_gazebo)/urdf/wamv_gazebo.xacro"/>
   <!-- === Batteries === -->
+  <!--
   <xacro:include filename="$(find wamv_description)/urdf/battery.xacro"/>
   <xacro:battery prefix="left" position="0 1 0.45" orientation="0 0 0"/>
   <xacro:battery prefix="right" position="0 -1 0.45" orientation="0 0 0"/>
+  -->
   <!-- === Thrusters === -->
   <!-- Use thruster yaml file if given -->

Commit message: feat: update WAM-V model with custom iacquabot meshes, adjust sensor positions, and add configurable spawn parameters to competition launch file

File: vrx_urdf/wamv_description/urdf/wamv_base.urdf.xacro (robot description, xacro)
@@ -86,8 +86,13 @@
   <!-- Basic model of the 16' WAM-V USV -->
   <link name="${namespace}/base_link">
-    <visual>
+    <!-- Main base hull (base.glb) -->
+    <visual name="base_visual">
+      <origin xyz="0 0 0.05" rpy="1.5708 0 3.14159"/>
       <geometry>
-        <mesh filename="package://wamv_description/models/WAM-V-Base/mesh/WAM-V-Base.dae"/>
+        <mesh filename="package://wamv_description/models/iacquabot_model/base.glb" scale="1.15 1.15 1.15"/>
       </geometry>
+      <material name="iacquabot_green">
+        <color rgba="0.18039 0.49020 0.19608 1.0"/>
+      </material>
     </visual>
     <!-- Left base collisions -->
@@ -108,4 +113,21 @@
     </inertial>
   </link>
+  <!-- Front Bow (proa.STL) as separate link for PBR metallic material support -->
+  <link name="${namespace}/proa_link">
+    <visual name="proa_visual">
+      <origin xyz="0 0 0" rpy="1.5708 0 1.5708"/>
+      <geometry>
+        <mesh filename="package://wamv_description/models/iacquabot_model/proa.STL" scale="0.001 0.001 0.001"/>
+      </geometry>
+      <material name="iacquabot_dark_blue">
+        <color rgba="0.015 0.065 0.320 1.0"/>
+      </material>
+    </visual>
+  </link>
+  <joint name="${namespace}/proa_joint" type="fixed">
+    <origin xyz="0.40 -0.22368 -0.02" rpy="0 0 0"/>
+    <parent link="${namespace}/base_link"/>
+    <child link="${namespace}/proa_link"/>
+  </joint>
   <gazebo>
     <enable_wind>true</enable_wind>
@@ -114,14 +136,7 @@
     <visual>
       <material>
-        <diffuse>1.0 1.0 1.0</diffuse>
-        <specular>1.0 1.0 1.0</specular>
-        <pbr>
-          <metal>
-            <albedo_map>model://wamv_description/models/WAM-V-Base/mesh/WAM-V_Albedo.png</albedo_map>
-            <normal_map>model://wamv_description/models/WAM-V-Base/mesh/WAM-V_Normal.png</normal_map>
-            <roughness_map>model://wamv_description/models/WAM-V-Base/mesh/WAM-V_Roughness.png</roughness_map>
-            <metalness_map>model://wamv_description/models/WAM-V-Base/mesh/WAM-V_Metalness.png</metalness_map>
-          </metal>
-        </pbr>
+        <ambient>0.18039 0.49020 0.19608 1.0</ambient>
+        <diffuse>0.18039 0.49020 0.19608 1.0</diffuse>
+        <specular>0.5 0.5 0.5 1.0</specular>
       </material>
     </visual>
@@ -142,3 +157,18 @@
     </sensor>
   </gazebo>
+  <gazebo reference="${namespace}/proa_link">
+    <visual>
+      <material>
+        <ambient>0.015 0.065 0.320 1.0</ambient>
+        <diffuse>0.015 0.065 0.320 1.0</diffuse>
+        <specular>1.0 1.0 1.0 1.0</specular>
+        <pbr>
+          <metal>
+            <roughness>0.15</roughness>
+            <metalness>0.9</metalness>
+          </metal>
+        </pbr>
+      </material>
+    </visual>
+  </gazebo>
 </robot>

File: vrx_urdf/wamv_gazebo/urdf/components/wamv_camera.xacro (robot description, xacro)
@@ -1,5 +1,5 @@
 <?xml version="1.0"?>
 <robot xmlns:xacro="http://ros.org/wiki/xacro">
-  <xacro:macro name="wamv_camera" params="name x:=0.5 y:=0 z:=1.5 post_z_from:=1.2965 R:=0 P:=0 Y:=0 post_Y:=0 visualize:=False">
+  <xacro:macro name="wamv_camera" params="name x:=0.30 y:=0 z:=0.40 post_z_from:=0.05 R:=0 P:=0 Y:=0 post_Y:=0 visualize:=False">
     <!-- Define length variables for link positioning -->
     <xacro:property name="platform_z" value="${post_z_from}"/>

File: vrx_urdf/wamv_gazebo/urdf/components/wamv_imu.xacro (robot description, xacro)
@@ -1,5 +1,5 @@
 <?xml version="1.0"?>
 <robot xmlns:xacro="http://ros.org/wiki/xacro">
-  <xacro:macro name="wamv_imu" params="name:=imu x:=0.3 y:=0.5 z:=1.3 R:=0 P:=0 Y:=0 update_rate:=100">
+  <xacro:macro name="wamv_imu" params="name:=imu x:=0.0 y:=0.0 z:=0.10 R:=0 P:=0 Y:=0 update_rate:=100">
     <link name="${namespace}/${name}_link">
       <visual name="${name}_visual">>

File: vrx_urdf/wamv_gazebo/urdf/wamv_gazebo.urdf.xacro (robot description, xacro)
@@ -106,5 +106,5 @@
     <!-- Add a front camera -->
     <xacro:if value="$(arg camera_enabled)">
-      <xacro:wamv_camera name="front_camera" y="0.3" x="0.75" P="${radians(15)}" />
+      <xacro:wamv_camera name="front_camera" x="0.30" y="0.0" z="0.40" post_z_from="0.05" P="${radians(15)}" />
     </xacro:if>
     <!-- Add simulated GPS -->
@@ -114,5 +114,5 @@
     <!-- Add Simulated IMU -->
     <xacro:if value="$(arg imu_enabled)">
-      <xacro:wamv_imu name="imu_wamv" y="-0.2" />
+      <xacro:wamv_imu name="imu_wamv" x="0.0" y="0.0" z="0.10" />
     </xacro:if>
     <!-- Add 3D LIDAR -->
@@ -145,5 +145,5 @@
       <xacro:wamv_gps name="gps_wamv" x="-0.85" />
       <!-- Add Simulated IMU -->
-      <xacro:wamv_imu name="imu_wamv" y="-0.2" />
+      <xacro:wamv_imu name="imu_wamv" x="0.0" y="0.0" z="0.10" />
       <!-- Add 3D LIDAR -->
       <xacro:lidar name="lidar_wamv" type="16_beam"/>

Commit message: add configuration

File: vrx_urdf/wamv_description/urdf/wamv_base.urdf.xacro (robot description, xacro)
@@ -105,9 +105,8 @@
       </geometry>
     </collision>
-    <inertial>
-      <!-- Customized WAM-V base values from user -->
-      <mass value="24.0"/>
-      <inertia ixx="4.77" ixy="0.0" ixz="0.0" iyy="1.01" iyz="0.0" izz="5.78"/>
-    </inertial>
+<inertial>
+  <mass value="21.92"/>
+  <inertia ixx="0.94" ixy="0.0" ixz="0.0" iyy="2.91" iyz="0.0" izz="2.59"/>
+</inertial>
   </link>
   <!-- Front Bow (proa.STL) as separate link for PBR metallic material support -->

File: vrx_urdf/wamv_gazebo/urdf/dynamics/wamv_gazebo_dynamics_plugin.xacro (robot description, xacro)
@@ -2,5 +2,5 @@
 <robot xmlns:xacro="http://ros.org/wiki/xacro">
   <xacro:macro name="usv_dynamics_gazebo" params="name wavefield_size:=1000">
-    <!--Gazebo Plugin for simulating WAM-V dynamics-->
+    <!--Gazebo Plugin for simulating board dynamics-->
     <gazebo>
       <!-- Left hull -->
@@ -9,10 +9,10 @@
         name="vrx::Surface">
         <link_name>${namespace}/base_link</link_name>
-        <hull_length>4.9</hull_length>
-        <hull_radius>0.213</hull_radius>
+        <hull_length>1.2</hull_length>
+        <hull_radius>0.15</hull_radius>
         <fluid_level>0</fluid_level>
         <points>
-          <point>0.6 1.03 0</point>
-          <point>-1.4 1.03 0</point>
+          <point>0.6 0.169 0</point>
+          <point>-0.6 0.169 0</point>
         </points>
         <wavefield>
@@ -25,10 +25,10 @@
         name="vrx::Surface">
         <link_name>${namespace}/base_link</link_name>
-        <hull_length>4.9</hull_length>
-        <hull_radius>0.213</hull_radius>
+        <hull_length>1.2</hull_length>
+        <hull_radius>0.15</hull_radius>
         <fluid_level>0</fluid_level>
         <points>
-          <point>0.6 -1.03 0</point>
-          <point>-1.4 -1.03 0</point>
+          <point>0.6 -0.169 0</point>
+          <point>-0.6 -0.169 0</point>
         </points>
         <wavefield>
@@ -36,24 +36,25 @@
         </wavefield>
       </plugin>
-      <plugin
+    <plugin
         filename="libSimpleHydrodynamics.so"
         name="vrx::SimpleHydrodynamics">
         <link_name>${namespace}/base_link</link_name>
         <!-- Added mass -->
-        <xDotU>0.0</xDotU>
-        <yDotV>0.0</yDotV>
-        <nDotR>0.0</nDotR>
-        <!-- Linear and quadratic drag -->
-        <xU>23.0</xU>
-        <xUU>38.0</xUU>
-        <yV>40.0</yV>
-        <yVV>30.0</yVV>
-        <zW>500.0</zW>
-        <kP>100.0</kP>
-        <kPP>100.0</kPP>
-        <mQ>100.0</mQ>
-        <mQQ>100.0</mQQ>
-        <nR>100.0</nR>
-        <nRR>10.0</nRR>
+        <xDotU>2.85</xDotU>
+        <yDotV>8.36</yDotV>
+        <nDotR>2.34</nDotR>
+        <!-- Arrastres Lineales y Cuadráticos Optimizados -->
+        <xU>13.91</xU>
+        <xUU>14.92</xUU>
+        <yV>49.04</yV>
+        <yVV>1.01</yVV>
+        <nR>6.03</nR>
+        <nRR>2.91</nRR>
+        <!-- ESTOS ERAN LOS CULPABLES (Bájalos drásticamente) -->
+        <zW>20.0</zW>    <!-- Fricción vertical (Heave) -->
+        <kP>2.0</kP>     <!-- Fricción de balanceo (Roll) -->
+        <kPP>2.0</kPP>
+        <mQ>5.0</mQ>     <!-- Fricción de cabeceo (Pitch) -->
+        <mQQ>5.0</mQQ>
       </plugin>
     </gazebo>

Commit message: no data yet

File: vrx_urdf/wamv_description/urdf/wamv_base.urdf.xacro (robot description, xacro)
@@ -103,5 +103,5 @@
 <inertial>
   <mass value="21.92"/>
-  <inertia ixx="0.94" ixy="0.0" ixz="0.0" iyy="2.91" iyz="0.0" izz="2.59"/>
+  <inertia ixx="0.94" ixy="0.0" ixz="0.0" iyy="2.91" iyz="0.0" izz="3.7"/>
 </inertial>
   </link>

File: vrx_urdf/wamv_gazebo/urdf/dynamics/wamv_gazebo_dynamics_plugin.xacro (robot description, xacro)
@@ -43,7 +43,7 @@
           name="vrx::SimpleHydrodynamics">
           <link_name>${namespace}/base_link</link_name>
-          <xDotU>2.85</xDotU>
-          <yDotV>8.36</yDotV>
-          <nDotR>1.957</nDotR>
+          <xDotU>1.426</xDotU>   <!-- ζ1 - m = 24.77 - 23.344 -->
+          <yDotV>6.936</yDotV>   <!-- ζ2 - m = 30.28 - 23.344 -->
+          <nDotR>2.006688</nDotR> <!-- ζ3 - Iz = 4.93 - 2.923312 -->
           <xU>13.91</xU>
           <xUU>14.92</xUU>
