Commit message: add cw and ccw propeller

File: vrx_urdf/wamv_gazebo/urdf/dynamics/wamv_gazebo_dynamics_plugin.xacro (robot description, xacro)
@@ -43,7 +43,7 @@
           name="vrx::SimpleHydrodynamics">
           <link_name>${namespace}/base_link</link_name>
-          <xDotU>-1.426</xDotU>   <!-- ζ1 - m = 24.77 - 23.344 -->
-          <yDotV>-6.936</yDotV>   <!-- ζ2 - m = 30.28 - 23.344 -->
-          <nDotR>-2.006688</nDotR> <!-- ζ3 - Iz = 4.93 - 2.923312 -->
+          <xDotU>1.426</xDotU>
+          <yDotV>6.936</yDotV>
+          <nDotR>2.006688</nDotR>
           <xU>13.91</xU>
           <xUU>14.92</xUU>

File: vrx_urdf/wamv_gazebo/urdf/thruster_layouts/wamv_aft_thrusters.xacro (robot description, xacro)
@@ -5,5 +5,5 @@
   <xacro:engine prefix="right" position="-0.10 -0.20 0.468237" />
   <xacro:include filename="$(find wamv_gazebo)/urdf/thruster_layouts/wamv_gazebo_thruster_config.xacro" />
-  <xacro:wamv_gazebo_thruster_config name="left" />
-  <xacro:wamv_gazebo_thruster_config name="right" />
+  <xacro:wamv_gazebo_thruster_config name="left" thrust_coefficient="0.1079" />
+  <xacro:wamv_gazebo_thruster_config name="right" thrust_coefficient="-0.1079" />
 </robot>

File: vrx_urdf/wamv_gazebo/urdf/thruster_layouts/wamv_gazebo_thruster_config.xacro (robot description, xacro)
@@ -1,5 +1,5 @@
 <?xml version="1.0"?>
 <plugin xmlns:xacro="http://ros.org/wiki/xacro">
-  <xacro:macro name="wamv_gazebo_thruster_config" params="name">
+  <xacro:macro name="wamv_gazebo_thruster_config" params="name thrust_coefficient:='0.1079'">
   <gazebo>
     <plugin
@@ -8,5 +8,5 @@
       <joint_name>${namespace}/${name}_engine_propeller_joint</joint_name>
       <cmd_timeout>0.5</cmd_timeout>
-      <thrust_coefficient>0.1079</thrust_coefficient>
+      <thrust_coefficient>${thrust_coefficient}</thrust_coefficient>
       <fluid_density>1000</fluid_density>
       <propeller_diameter>0.0762</propeller_diameter>

File: vrx_urdf/wamv_gazebo/urdf/thruster_layouts/wamv_t_thrusters.xacro (robot description, xacro)
@@ -6,6 +6,6 @@
   <xacro:engine prefix="lateral" position="0.60 0.0 0.468237" orientation="0.0 0.0 1.5707"/>
   <xacro:include filename="$(find wamv_gazebo)/urdf/thruster_layouts/wamv_gazebo_thruster_config.xacro" />
-  <xacro:wamv_gazebo_thruster_config name="left" />
-  <xacro:wamv_gazebo_thruster_config name="right" />
-  <xacro:wamv_gazebo_thruster_config name="lateral" />
+  <xacro:wamv_gazebo_thruster_config name="left" thrust_coefficient="0.1079" />
+  <xacro:wamv_gazebo_thruster_config name="right" thrust_coefficient="-0.1079" />
+  <xacro:wamv_gazebo_thruster_config name="lateral" thrust_coefficient="0.1079" />
 </robot>

File: vrx_urdf/wamv_gazebo/urdf/thruster_layouts/wamv_x_thrusters.xacro (robot description, xacro)
@@ -7,7 +7,7 @@
   <xacro:engine prefix="right_front" position=" 0.60 -0.29 0.468237" orientation="0.0 0.0 0.0"/>
   <xacro:include filename="$(find wamv_gazebo)/urdf/thruster_layouts/wamv_gazebo_thruster_config.xacro" />
-  <xacro:wamv_gazebo_thruster_config name="left_rear" />
-  <xacro:wamv_gazebo_thruster_config name="right_rear" />
-  <xacro:wamv_gazebo_thruster_config name="left_front" />
-  <xacro:wamv_gazebo_thruster_config name="right_front" />
+  <xacro:wamv_gazebo_thruster_config name="left_rear" thrust_coefficient="0.1079" />
+  <xacro:wamv_gazebo_thruster_config name="right_rear" thrust_coefficient="-0.1079" />
+  <xacro:wamv_gazebo_thruster_config name="left_front" thrust_coefficient="0.1079" />
+  <xacro:wamv_gazebo_thruster_config name="right_front" thrust_coefficient="-0.1079" />
 </robot>
